File: starfish/led-driver.kicad_sch (KiCad schematic)
At the start: 16 parts, among them Q50 PMV40UN2R, Q52 PMV40UN2R, Q54 PMV40UN2R, Q56 PMV40UN2R, Q58 PMV40UN2R

Commit message: Start rev b
Parts:
- removed JP58: CH5, Jumper:SolderJumper-2_P1.3mm_Open_RoundedPad1.0x1.5mm, symbol Jumper:SolderJumper_2_Open
- removed Q58: PMV40UN2R, Package_TO_SOT_SMD:SOT-23, symbol paeber:PMV40UN2R
- removed R58: 330, Resistor_SMD:R_0603_1608Metric_Pad0.98x0.95mm_HandSolder, symbol Device:R
- removed R59: 10k, Resistor_SMD:R_0603_1608Metric_Pad0.98x0.95mm_HandSolder, symbol Device:R
