File: starfish/power.kicad_sch (KiCad schematic)
At the start: 14 parts, among them U20 AP62301WU-7

Commit message: Start rev b
Connections:
- net 5V renamed V_REG
Other:
- note added: "R23 = 4k7 for 3V3 output"

Commit message: Layout progress
Parts:
- C20: Mouser 603-AC0805KR9BB104 -> 581-06035C104KAT2A
Changed lines of the file:
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@@
       (effects (font (size 1.27 1.27)) hide)
     )
-    (property "Mouser" "603-AC0805KR9BB104" (at 143.51 60.96 0)
+    (property "Mouser" "581-06035C104KAT2A" (at 143.51 60.96 0)
       (effects (font (size 1.27 1.27)) hide)
     )
