File: starfish/starfish.kicad_pcb (KiCad board)
At the start: 2 copper layers, 60 x 50 mm, 65 parts, among them J1 USB4105-GF-A-120, J10 UartBridge, J2 Barrel_Jack_Switch, J3 Screw_Terminal_01x02, J90 Screw_Terminal_01x06, Q12 BSS138, Q14 BSS138, Q50 PMV40UN2R, Q52 PMV40UN2R, Q54 PMV40UN2R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

Commit message: Start rev b
Parts:
- removed JP58: CH5, Jumper:SolderJumper-2_P1.3mm_Open_RoundedPad1.0x1.5mm
- removed Q58: PMV40UN2R, Package_TO_SOT_SMD:SOT-23
- removed R58: 330, Resistor_SMD:R_0603_1608Metric_Pad0.98x0.95mm_HandSolder
- removed R59: 10k, Resistor_SMD:R_0603_1608Metric_Pad0.98x0.95mm_HandSolder
- added J4: Conn_02x02_Odd_Even, Connector_PinHeader_2.54mm:PinHeader_2x02_P2.54mm_Vertical, F.Cu at (155.9, 49.3)
- added J5: Conn_02x02_Odd_Even, Connector_PinHeader_2.54mm:PinHeader_2x02_P2.54mm_Vertical, F.Cu at (122.2, 86.8)
- added JP1: SolderJumper_2_Open, Jumper:SolderJumper-2_P1.3mm_Open_RoundedPad1.0x1.5mm, F.Cu at (140.4, 48.5)
- added JP2: SolderJumper_2_Open, Jumper:SolderJumper-2_P1.3mm_Open_RoundedPad1.0x1.5mm, F.Cu at (140.4, 52.0)
- J3: footprint TerminalBlock:TerminalBlock_bornier-2_P5.08mm -> paeber:CUI_TBP01R1-508-02BE
- J90: footprint TerminalBlock:TerminalBlock_bornier-6_P5.08mm -> paeber:CUI_TBP01R1-508-06BE
- SW10, SW11, SW60: value TS-1095PS-A3B3-C3D2 -> 1301.9315; footprint Button_Switch_SMD:SW_SPST_PTS645 -> paeber:13019319
- moved J90 25.7 mm to (176.2, 72.0), turned to -90 degrees
- moved SW11 6.50 mm to (133.2, 100.0)
- moved R13 5.12 mm to (132.6, 94.0)
- moved J3 4.32 mm to (123.6, 77.2), turned to 90 degrees
- moved SW60 2.20 mm to (162.2, 64.0)
- moved SW10 2.03 mm to (148.1, 100.0)
- moved H3 0.19 mm to (175.0, 105.0)
- moved H4 0.19 mm to (175.0, 65.0)
Connections:
- C22 pad 1: +5V -> /Power/V_REG
- C23 pad 1: +5V -> /Power/V_REG
- J90 pad 1: /LED Driver/PWM1 -> GND
- J90 pad 2: /LED Driver/PWM2 -> Net-(J90-Pin_2)
- J90 pad 3: /LED Driver/PWM3 -> /LED Driver/PWM4
- J90 pad 4: /LED Driver/PWM4 -> /LED Driver/PWM3
- J90 pad 5: /LED Driver/PWM5 -> /LED Driver/PWM2
- J90 pad 6: Net-(J90-Pad6) -> /LED Driver/PWM1
- JP90 pad 2: Net-(J90-Pad6) -> Net-(J90-Pin_2)
- L20 pad 2: +5V -> /Power/V_REG
- R22 pad 1: +5V -> /Power/V_REG
- TP22 pad 1: +5V -> /Power/V_REG
- U10 pad 18: /CH5 -> unconnected-(U10-GPIO10/TOUCH10/ADC1_CH9/FSPICS0/FSPIIO4/SUBSPICS0-Pad18)
Routing:
- net VCC: track 104.4 -> 71.9 mm
- net /CH5: track 25.9 -> 0.00 mm, vias 1 -> 0
- net /LED Driver/PWM5: track 18.6 -> 0.00 mm
- net unconnected-(U10-GPIO10/TOUCH10/ADC1_CH9/FSPICS0/FSPIIO4/SUBSPICS0-Pad18): track 0.00 -> 16.5 mm, vias 0 -> 1
- net /GPIO0: track 35.4 -> 26.8 mm
- net Net-(JP58-Pad1): track 8.22 -> 0.00 mm, vias 1 -> 0
- net Net-(J90-Pad6): track 6.04 -> 0.00 mm
- net GND: track 45.2 -> 41.5 mm, vias 75 -> 71
- net /CHIP_PU: track 24.2 -> 20.5 mm
- net +5V: track 118.0 -> 117.0 mm
Other:
- board text removed: "PaEber"

Commit message: Add some components
Parts:
- removed J5: Conn_02x02_Odd_Even, Connector_PinHeader_2.54mm:PinHeader_2x02_P2.54mm_Vertical
- added J6: Conn_01x04, Connector_PinSocket_2.54mm:PinSocket_1x04_P2.54mm_Vertical, F.Cu at (218.6, 90.8)
- added J7: Conn_01x04, Connector_PinSocket_2.54mm:PinSocket_1x04_P2.54mm_Vertical, F.Cu at (212.4, 50.0)
- added J9: Conn_01x04, Connector_PinSocket_2.54mm:PinSocket_1x04_P2.54mm_Vertical, F.Cu at (108.0, 53.8)
- added R3: 10k, Resistor_SMD:R_0603_1608Metric_Pad0.98x0.95mm_HandSolder, F.Cu at (240.0, 77.0)
- added SW61: 1301.9315, paeber:13019319, F.Cu at (222.2, 80.3)
- J4: value Conn_02x02_Odd_Even -> Conn_01x04; footprint Connector_PinHeader_2.54mm:PinHeader_2x02_P2.54mm_Vertical -> Connector_PinSocket_2.54mm:PinSocket_1x04_P2.54mm_Vertical
- moved J4 4.60 mm to (157.0, 53.8), turned to 180 degrees
- moved J2 0.85 mm to (133.0, 73.4)
Connections:
- J4 pad 1: +5V -> VCC
- J4 pad 3: GND -> +3V3
- U10 pad 18: unconnected-(U10-GPIO10/TOUCH10/ADC1_CH9/FSPICS0/FSPIIO4/SUBSPICS0-Pad18) -> /I2C_SCL
- U10 pad 19: /CH4 -> /I2C_SDA
- U10 pad 20: /CH3 -> /GPIO12
- U10 pad 21: /CH2 -> /GPIO13
- U10 pad 22: /CH1 -> /GPIO14
- U10 pad 26: unconnected-(U10-GPIO45-Pad26) -> Net-(SW61-A)
- U10 pad 4: unconnected-(U10-GPIO4/TOUCH4/ADC1_CH3-Pad4) -> /CH4
- U10 pad 5: unconnected-(U10-GPIO5/TOUCH5/ADC1_CH4-Pad5) -> /CH3
- U10 pad 6: unconnected-(U10-GPIO6/TOUCH6/ADC1_CH5-Pad6) -> /CH2
- U10 pad 7: unconnected-(U10-GPIO7/TOUCH7/ADC1_CH6-Pad7) -> /CH1
Routing:
- net unconnected-(U10-GPIO10/TOUCH10/ADC1_CH9/FSPICS0/FSPIIO4/SUBSPICS0-Pad18): track 16.5 -> 0.00 mm, vias 1 -> 0
- net /I2C_SCL: track 0.00 -> 16.5 mm, vias 0 -> 1

Commit message: Power progress
Parts:
- removed GPIO1: TestPoint, TestPoint:TestPoint_Pad_D2.5mm
- added J5: Conn_02x02_Odd_Even, Connector_PinHeader_2.54mm:PinHeader_2x02_P2.54mm_Vertical, F.Cu at (131.0, 75.0)
- added J8: Conn_02x02_Odd_Even, Connector_PinHeader_2.54mm:PinHeader_2x02_P2.54mm_Vertical, F.Cu at (125.0, 86.0)
- added JP3: SolderJumper_3_Open, Jumper:SolderJumper-3_P1.3mm_Open_RoundedPad1.0x1.5mm, B.Cu at (131.5, 64.5)
- C1, C2, C3, U1: moved to B.Cu
- moved SW61 63.9 mm to (159.5, 67.6), turned to 90 degrees
- moved J6 32.7 mm to (232.5, 61.2)
- moved J4 28.2 mm to (130.0, 62.0), turned to 90 degrees
- moved C3 25.7 mm to (142.5, 65.0), turned to -90 degrees
- moved J7 20.9 mm to (191.5, 48.7)
- moved JP1 18.3 mm to (132.5, 65.0), turned to 90 degrees
- moved U1 18.0 mm to (137.5, 67.5), turned to 90 degrees
- moved C1 14.6 mm to (131.0, 67.0)
- moved C2 14.6 mm to (131.0, 69.5), turned to 180 degrees
- moved JP2 14.1 mm to (135.0, 65.0), turned to 90 degrees
- moved C22 6.36 mm to (134.0, 68.0), turned to 180 degrees
- moved SW60 5.81 mm to (167.6, 66.0), turned to -90 degrees
- moved J2 5.29 mm to (128.0, 75.2)
- moved TP22 4.70 mm to (138.7, 65.0)
- moved D1 2.20 mm to (128.0, 87.0)
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Connections:
- C1 pad 1: +5V -> /VIN_LIN
- C2 pad 1: +5V -> /VIN_LIN
- J3 pad 1: VCC -> GND
- J3 pad 2: GND -> VCC
- U1 pad 3: +5V -> /VIN_LIN
- U10 pad 16: unconnected-(U10-GPIO46-Pad16) -> Net-(SW60-A)
- U10 pad 23: Net-(SW60-A) -> unconnected-(U10-GPIO21-Pad23)
- U10 pad 39: Net-(U10-GPIO1/TOUCH1/ADC1_CH0) -> unconnected-(U10-GPIO1/TOUCH1/ADC1_CH0-Pad39)
Routing:
- net Net-(SW60-A): track 36.3 -> 0.00 mm, vias 2 -> 0
- net /CH1: track 26.8 -> 0.00 mm, vias 1 -> 0
- net /CH3: track 25.9 -> 0.00 mm, vias 1 -> 0
- net /CH2: track 25.3 -> 0.00 mm, vias 1 -> 0
- net /CH4: track 24.5 -> 0.21 mm, vias 1 -> 0
- net Net-(Q12-D): track 31.1 -> 7.32 mm
- net +5V: track 117.0 -> 93.6 mm, vias 8 -> 1
- net GND: track 41.5 -> 23.5 mm, vias 71 -> 48
- net /I2C_SCL: track 16.5 -> 0.00 mm, vias 1 -> 0
- net Net-(U10-GPIO1/TOUCH1/ADC1_CH0): track 10.3 -> 0.00 mm, vias 1 -> 0
- net VCC: track 71.9 -> 80.8 mm
- net /VIN_LIN: track 0.00 -> 8.86 mm
- net /CHIP_PU: track 20.5 -> 13.8 mm
- net Net-(Q52-G): track 4.73 -> 0.06 mm
- net Net-(Q12-G): track 9.67 -> 8.58 mm
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- added copper zone on F.Cu, net /Power/V_REG
- removed copper zone on F.Cu, net +3V3
- removed copper zone on B.Cu, net +5V
- removed copper zone on F.Cu, net +5V

Commit message: Rev b progress
Parts:
- removed G***: LOGO, LOGO
- added D2: PMEG60T10ELRX, Diode_SMD:D_SOD-123, F.Cu at (130.5, 85.5)
- Q12: moved to B.Cu
- SW10, SW11: value 1301.9315 -> PTS636SK25; footprint paeber:13019319 -> Button_Switch_SMD:SW_Tactile_SPST_NO_Straight_CK_PTS636Sx25SMTRLFS
- moved J6 103.3 mm to (131.0, 80.0), turned to 90 degrees
- moved R3 100.0 mm to (140.5, 87.0)
- moved J7 40.5 mm to (154.0, 64.0)
- moved R13 12.7 mm to (143.5, 100.5), turned to 0 degrees
- moved R11 10.7 mm to (143.5, 102.0), turned to 0 degrees
- moved JP90 7.67 mm to (169.5, 62.5)
- moved SW11 7.21 mm to (139.5, 96.5), turned to -90 degrees
- moved R60 5.88 mm to (140.5, 88.5), turned to 0 degrees
- moved C11 5.70 mm to (130.0, 101.5), turned to -90 degrees
- moved R10 5.20 mm to (146.5, 90.0)
- moved Q12 4.34 mm to (165.5, 95.0), turned to 180 degrees
- moved SW10 3.55 mm to (147.5, 96.5), turned to 90 degrees
- moved D1 1.50 mm to (128.0, 85.5)
- moved TP20 1.50 mm to (142.5, 76.5)
- moved SW61 0.99 mm to (160.5, 67.5)
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Connections:
- net /USB_DM renamed /USB_DN
- J8 pad 1: +5V -> +3V3
- J8 pad 3: +3V3 -> +5V
- R3 pad 1: Net-(SW61-A) -> /BTN_2
- R60 pad 1: Net-(SW60-A) -> /BTN_1
- SW10 pad 1: /GPIO0 -> GND
- SW10 pad 2: GND -> /GPIO0
- SW11 pad 1: /CHIP_PU -> GND
- SW11 pad 2: GND -> /CHIP_PU
- SW60 pad 1: Net-(SW60-A) -> /BTN_1
- SW61 pad 1: Net-(SW61-A) -> /BTN_2
- U10 pad 12: unconnected-(U10-GPIO8/TOUCH8/ADC1_CH7/SUBSPICS1-Pad12) -> /BTN_1
- U10 pad 16: Net-(SW60-A) -> unconnected-(U10-GPIO46-Pad16)
- U10 pad 17: unconnected-(U10-GPIO9/TOUCH9/ADC1_CH8/FSPIHD/SUBSPIHD-Pad17) -> /I2C_SCL
- U10 pad 18: /I2C_SCL -> /I2C_SDA
- U10 pad 19: /I2C_SDA -> /BTN_2
- U10 pad 26: Net-(SW61-A) -> unconnected-(U10-GPIO45-Pad26)
- U10 pad 4: /CH4 -> /CH1
- U10 pad 5: /CH3 -> /CH2
- U10 pad 6: /CH2 -> /CH3
- U10 pad 7: /CH1 -> /CH4
Routing:
- net /CH4: track 0.21 -> 38.0 mm, vias 0 -> 1
- net /CH3: track 0.00 -> 33.7 mm, vias 0 -> 1
- net /CH2: track 0.00 -> 30.7 mm, vias 0 -> 1
- net /CH1: track 0.00 -> 29.1 mm, vias 0 -> 1
- net Net-(J90-Pin_2): track 0.00 -> 25.9 mm
- net /GPIO12: track 0.00 -> 16.2 mm
- net /GPIO0: track 26.8 -> 10.8 mm, vias 2 -> 1
- net Net-(Q12-D): track 7.32 -> 23.3 mm, vias 0 -> 1
- net /GPIO13: track 0.00 -> 14.6 mm
- net GND: track 23.5 -> 9.97 mm, vias 48 -> 15
- net /GPIO14: track 0.00 -> 12.9 mm
- net +5V: track 93.6 -> 83.2 mm
- net /I2C_SCL: track 0.00 -> 6.94 mm
- net /I2C_SDA: track 0.00 -> 5.58 mm
- net /Power/FB_5V: track 5.29 -> 0.00 mm
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Other:
- board text removed: "Starfish Rev A"

Commit message: Layout progress
Parts:
- removed J9: Conn_01x04, Connector_PinSocket_2.54mm:PinSocket_1x04_P2.54mm_Vertical
- added J11: Conn_01x03, Connector_PinSocket_2.54mm:PinSocket_1x03_P2.54mm_Vertical, F.Cu at (162.0, 77.0)
- added J65: Conn_01x02, Connector_PinHeader_2.54mm:PinHeader_1x02_P2.54mm_Vertical, F.Cu at (172.0, 70.7)
- added R4: 4k7, Resistor_SMD:R_0603_1608Metric_Pad0.98x0.95mm_HandSolder, F.Cu at (140.5, 88.0)
- added R5: 4k7, Resistor_SMD:R_0603_1608Metric_Pad0.98x0.95mm_HandSolder, F.Cu at (142.0, 88.0)
- added R65: 10k, Resistor_SMD:R_0603_1608Metric_Pad0.98x0.95mm_HandSolder, B.Cu at (156.5, 66.5)
- added U65: LTV-817S, Package_DIP:SMDIP-4_W9.53mm, B.Cu at (164.0, 68.5)
- C10, C11: footprint Capacitor_SMD:C_0805_2012Metric_Pad1.18x1.45mm_HandSolder -> Capacitor_SMD:C_0603_1608Metric_Pad1.08x0.95mm_HandSolder; moved to F.Cu
- C12: footprint Capacitor_SMD:C_0805_2012Metric_Pad1.18x1.45mm_HandSolder -> Capacitor_SMD:C_0603_1608Metric_Pad1.08x0.95mm_HandSolder
- moved C10 11.2 mm to (146.5, 87.0), turned to 180 degrees
- moved C11 9.51 mm to (139.5, 102.0), turned to 180 degrees
- moved SW60 9.01 mm to (159.0, 66.5)
- moved R15 8.79 mm to (165.5, 93.5)
- moved SW61 6.02 mm to (166.5, 68.0)
- moved R3 3.16 mm to (143.5, 88.0), turned to -90 degrees
- moved R51 3.11 mm to (166.5, 97.5)
- moved R53 3.11 mm to (166.5, 93.5)
- moved R55 3.11 mm to (166.5, 89.5)
- moved R57 3.11 mm to (166.5, 85.5)
- moved R54 3.06 mm to (164.5, 89.5)
- moved R56 3.06 mm to (164.5, 85.5)
- moved Q54 3.04 mm to (169.5, 89.5)
- moved Q56 3.04 mm to (169.5, 85.5)
- moved R50 3.04 mm to (164.5, 97.5)
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Routing:
- net +3V3: track 33.5 -> 120.9 mm, vias 0 -> 1
- net /BTN_1: track 0.00 -> 46.6 mm, vias 0 -> 1
- net /BTN_2: track 0.00 -> 42.9 mm, vias 0 -> 1
- net /GPIO0: track 10.8 -> 29.8 mm, vias 1 -> 2
- net Net-(Q14-D): track 11.7 -> 2.15 mm
- net /Power/V_REG: track 0.00 -> 8.80 mm, vias 0 -> 2
- net /CHIP_PU: track 15.5 -> 8.37 mm
- net /Power/FB_5V: track 0.00 -> 6.59 mm
- net /GPIO12: track 16.2 -> 20.7 mm
- net Net-(Q52-G): track 0.06 -> 4.08 mm
- net /GPIO13: track 14.6 -> 17.6 mm
- net /I2C_SDA: track 5.58 -> 8.49 mm, vias 0 -> 1
- net /I2C_SCL: track 6.94 -> 9.80 mm, vias 0 -> 1
- net /AIN_TTL: track 0.00 -> 2.81 mm
- net /CH4: track 38.0 -> 35.4 mm
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Other:
- board text removed: "GP10"

Commit message: RevB first gerber export
Parts:
- added C4: 100n, Capacitor_SMD:C_0603_1608Metric_Pad1.08x0.95mm_HandSolder, F.Cu at (151.0, 90.5)
- added D4: SK6812, LED_SMD:LED_SK6812_PLCC4_5.0x5.0mm_P3.2mm, F.Cu at (152.0, 86.5)
- added D65: PMEG60T10ELRX, Diode_SMD:D_SOD-123, B.Cu at (168.5, 67.0)
- added R66: 10k, Resistor_SMD:R_0603_1608Metric_Pad0.98x0.95mm_HandSolder, B.Cu at (169.5, 73.0)
- added REF**: KiCad-Logo2_5mm_SilkScreen, Symbol:KiCad-Logo2_5mm_SilkScreen, B.Cu at (167.5, 81.5)
- moved U65 3.61 mm to (162.0, 71.5)
- moved R2 0.50 mm to (130.5, 92.5)
Connections:
- J65 pad 1: Net-(J65-Pin_1) -> Net-(D65-A)
- J7 pad 2: /GPIO12 -> /AIN_TTL
- U10 pad 20: /GPIO12 -> /AIN_TTL
- U10 pad 31: unconnected-(U10-GPIO38/FSPIWP/SUBSPIWP-Pad31) -> /LED_DIN
- U65 pad 1: Net-(J65-Pin_1) -> Net-(D65-K)
- U65 pad 2: Net-(J65-Pin_2) -> Net-(R66-Pad2)
Routing:
- net +3V3: track 120.9 -> 146.3 mm, vias 1 -> 3
- net /AIN_TTL: track 2.81 -> 26.4 mm
- net /GPIO12: track 20.7 -> 0.00 mm
- net /LED_DIN: track 0.00 -> 6.48 mm, vias 0 -> 1
- net Net-(D65-A): track 0.00 -> 4.70 mm
- net Net-(D65-K): track 0.00 -> 3.27 mm
- net Net-(R66-Pad2): track 0.00 -> 3.02 mm
- net Net-(J65-Pin_2): track 0.00 -> 2.77 mm
- net /CHIP_PU: track 8.37 -> 10.6 mm
- net GND: vias 6 -> 59
Other:
- board text added: "12"
- board text added: "13"
- board text added: "14"
- board text added: "5V"
- board text added: "BOOT"
- board text added: "GP3"
- board text added: "GP4"
- board text added: "GP5"
- board text added: "GP6"
- board text added: "GP8"
- board text added: "PaEber"
- board text added: "RESET"
- board text added: "SCL"
- board text added: "SDA"
- board text added: "Starfish Rev B PaEber 03/23"
- board text removed: "GP12"
- board text removed: "GP13"
- board text removed: "GP14"
