File: starfish/starfish.kicad_sch (KiCad schematic)
At the start: 34 parts, among them J1 USB4105-GF-A-120, J10 UartBridge, J2 Barrel_Jack_Switch, J3 Screw_Terminal_01x02, J90 Screw_Terminal_01x06, Q12 BSS138, Q14 BSS138, SW10 TS-1095PS-A3B3-C3D2, SW11 TS-1095PS-A3B3-C3D2, SW60 TS-1095PS-A3B3-C3D2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

Commit message: Start rev b
Parts:
- removed SW10, SW11, SW60: TS-1095PS-A3B3-C3D2, Button_Switch_SMD:SW_SPST_PTS645, symbol Switch:SW_SPST
- added J4, J5: Conn_02x02_Odd_Even, Connector_PinHeader_2.54mm:PinHeader_2x02_P2.54mm_Vertical, symbol Connector_Generic:Conn_02x02_Odd_Even
- added JP1, JP2: SolderJumper_2_Open, Jumper:SolderJumper-2_P1.3mm_Open_RoundedPad1.0x1.5mm, symbol Jumper:SolderJumper_2_Open
- added R3: 10k, Resistor_SMD:R_0603_1608Metric_Pad0.98x0.95mm_HandSolder, symbol Device:R
- added SW10, SW11, SW60, SW61: 1301.9315, paeber:13019319, symbol paeber:1301.9315
- J3: footprint TerminalBlock:TerminalBlock_bornier-2_P5.08mm -> paeber:CUI_TBP01R1-508-02BE
- J90: footprint TerminalBlock:TerminalBlock_bornier-6_P5.08mm -> paeber:CUI_TBP01R1-508-06BE
Connections:
- net LED Driver/PWM5 is gone; now on net LED Driver/PWM2: J90.5 (Pin_5)
- net +3V3: now also JP2.2 (B), R3.2
- net +5V: now also J4.1 (Pin_1), J4.2 (Pin_2), JP1.2 (B)
- net CHIP_PU: now also SW11.1 (A)
- net GND: now also J90.1 (Pin_1), J4.3 (Pin_3), J4.4 (Pin_4), J5.3 (Pin_3), J5.4 (Pin_4), SW10.2 (B), SW11.2 (B), SW60.2 (B), SW61.2 (B)
- net GPIO0: now also SW10.1 (A)
- net LED Driver/PWM1: now also J90.6 (Pin_6); no longer J90.1 (Pin_1)
- net LED Driver/PWM2: no longer J90.2 (Pin_2)
- net LED Driver/PWM3: now also J90.4 (Pin_4); no longer J90.3 (Pin_3)
- net LED Driver/PWM4: now also J90.3 (Pin_3); no longer J90.4 (Pin_4)
- net VCC: now also J5.1 (Pin_1), J5.2 (Pin_2)
- net at JP90.2 (C): now also J90.2 (Pin_2); no longer J90.6 (Pin_6)
- net at R60.1, U10.23 (GPIO21): now also SW60.1 (A)
- net at U10.26 (GPIO45): now also R3.1, SW61.1 (A)
- net CH5: no longer names the net of U10.18 (GPIO10/TOUCH10/ADC1_CH9/FSPICS0/FSPIIO4/SUBSPICS0)
- new net Power/V_REG: JP1.1 (A), JP2.1 (A)
Other:
- sheet LED Driver ports: added none; removed CH5, PWM5
- sheet Power ports: added V_REG; removed 5V
- note added: "GPIO0 GPIO2 GPIO4 GPIO12 GPIO13 GPIO14 GPIO15 GPIO27 GPIO32 GPIO33"

Commit message: Add some components
Parts:
- removed J4, J5: Conn_02x02_Odd_Even, Connector_PinHeader_2.54mm:PinHeader_2x02_P2.54mm_Vertical, symbol Connector_Generic:Conn_02x02_Odd_Even
- added J4, J6, J7, J9: Conn_01x04, Connector_PinSocket_2.54mm:PinSocket_1x04_P2.54mm_Vertical, symbol Connector_Generic:Conn_01x04
Connections:
- net +3V3: now also J4.3 (Pin_3), J6.2 (Pin_2), J9.1 (Pin_1)
- net +5V: now also J4.2 (Pin_2), J9.2 (Pin_2)
- net CH1: now also U10.7 (GPIO7/TOUCH7/ADC1_CH6); no longer U10.22 (GPIO14/TOUCH14/ADC2_CH3/FSPIWP/FSPIDQS/SUBSPIWP)
- net CH2: now also U10.6 (GPIO6/TOUCH6/ADC1_CH5); no longer U10.21 (GPIO13/TOUCH13/ADC2_CH2/FSPIQ/FSPIIO7/SUBSPIQ)
- net CH3: now also U10.5 (GPIO5/TOUCH5/ADC1_CH4); no longer U10.20 (GPIO12/TOUCH11/ADC2_CH0/FSPICS0/FSPIIO4/SUBSPICS0)
- net CH4: now also U10.4 (GPIO4/TOUCH4/ADC1_CH3); no longer U10.19 (GPIO11/TOUCH11/ADC2_CH0/FSPICS0/FSPIIO4/SUBSPICS0)
- net GND: now also J4.4 (Pin_4), J6.1 (Pin_1), J7.1 (Pin_1), J9.3 (Pin_3), J9.4 (Pin_4)
- net VCC: now also J4.1 (Pin_1)
- net I2C_SCL: now reaches U10.18 (GPIO10/TOUCH10/ADC1_CH9/FSPICS0/FSPIIO4/SUBSPICS0)
- net I2C_SCL: now also J6.3 (Pin_3)
- new net GPIO12: J7.2 (Pin_2), U10.20 (GPIO12/TOUCH11/ADC2_CH0/FSPICS0/FSPIIO4/SUBSPICS0)
- new net GPIO13: J7.3 (Pin_3), U10.21 (GPIO13/TOUCH13/ADC2_CH2/FSPIQ/FSPIIO7/SUBSPIQ)
- new net GPIO14: J7.4 (Pin_4), U10.22 (GPIO14/TOUCH14/ADC2_CH3/FSPIWP/FSPIDQS/SUBSPIWP)
- new net I2C_SDA: J6.4 (Pin_4), U10.19 (GPIO11/TOUCH11/ADC2_CH0/FSPICS0/FSPIIO4/SUBSPICS0)

Commit message: Power progress
Parts:
- removed GPIO1: TestPoint, TestPoint:TestPoint_Pad_D2.5mm, symbol Connector:TestPoint
- added J5, J8: Conn_02x02_Odd_Even, Connector_PinHeader_2.54mm:PinHeader_2x02_P2.54mm_Vertical, symbol Connector_Generic:Conn_02x02_Odd_Even
- added JP3: SolderJumper_3_Open, Jumper:SolderJumper-3_P1.3mm_Open_RoundedPad1.0x1.5mm, symbol Jumper:SolderJumper_3_Open
Connections:
- net +3V3: now also J8.3 (Pin_3)
- net +5V: now also J8.1 (Pin_1), JP3.1 (A); no longer C1.1, C2.1, U1.3 (VI)
- net GND: now also J3.1 (Pin_1), J5.2 (Pin_2), J5.4 (Pin_4), J8.2 (Pin_2), J8.4 (Pin_4); no longer J3.2 (Pin_2)
- net VCC: now also J3.2 (Pin_2), J5.1 (Pin_1), J5.3 (Pin_3), JP3.3 (B); no longer J3.1 (Pin_1)
- net at R60.1, SW60.1 (A): now also U10.16 (GPIO46); no longer U10.23 (GPIO21)
- new net VIN_LIN: C1.1, C2.1, JP3.2 (C), U1.3 (VI)
Other:
- moved on the sheet: J3, SW60

Commit message: Rev b progress
Parts:
- removed SW10, SW11: 1301.9315, paeber:13019319, symbol paeber:1301.9315
- added D2: PMEG60T10ELRX, Diode_SMD:D_SOD-123, symbol Device:D
- added SW10, SW11: PTS636SK25, Button_Switch_SMD:SW_Tactile_SPST_NO_Straight_CK_PTS636Sx25SMTRLFS, symbol Switch:SW_Push
Connections:
- net +3V3: now also J8.1 (Pin_1); no longer J8.3 (Pin_3)
- net +5V: now also J8.3 (Pin_3); no longer J8.1 (Pin_1)
- net CH1: now also U10.4 (GPIO4/TOUCH4/ADC1_CH3); no longer U10.7 (GPIO7/TOUCH7/ADC1_CH6)
- net CH2: now also U10.5 (GPIO5/TOUCH5/ADC1_CH4); no longer U10.6 (GPIO6/TOUCH6/ADC1_CH5)
- net CH3: now also U10.6 (GPIO6/TOUCH6/ADC1_CH5); no longer U10.5 (GPIO5/TOUCH5/ADC1_CH4)
- net CH4: now also U10.7 (GPIO7/TOUCH7/ADC1_CH6); no longer U10.4 (GPIO4/TOUCH4/ADC1_CH3)
- net CHIP_PU: now also SW11.2
- net GND: now also SW10.1, SW11.1
- net GPIO0: now also SW10.2
- net I2C_SCL: now also U10.17 (GPIO9/TOUCH9/ADC1_CH8/FSPIHD/SUBSPIHD); no longer U10.18 (GPIO10/TOUCH10/ADC1_CH9/FSPICS0/FSPIIO4/SUBSPICS0)
- net I2C_SDA: now also U10.18 (GPIO10/TOUCH10/ADC1_CH9/FSPICS0/FSPIIO4/SUBSPICS0); no longer U10.19 (GPIO11/TOUCH11/ADC2_CH0/FSPICS0/FSPIIO4/SUBSPICS0)
- net VBUS: now also D2.2 (A)
- net VCC: now also D2.1 (K)
- net BTN_1: now reaches R60.1, SW60.1 (A)
- net BTN_1: now also U10.12 (GPIO8/TOUCH8/ADC1_CH7/SUBSPICS1); no longer U10.16 (GPIO46)
- net BTN_2: now reaches R3.1, SW61.1 (A)
- net BTN_2: now also U10.19 (GPIO11/TOUCH11/ADC2_CH0/FSPICS0/FSPIIO4/SUBSPICS0); no longer U10.26 (GPIO45)
- net USB_DM renamed USB_DN
- no-connect marks 2 -> 5
Other:
- moved on the sheet: R3, R60, SW60, SW61

Commit message: Layout progress
Parts:
- removed J9: Conn_01x04, Connector_PinSocket_2.54mm:PinSocket_1x04_P2.54mm_Vertical, symbol Connector_Generic:Conn_01x04
- added J11: Conn_01x03, Connector_PinSocket_2.54mm:PinSocket_1x03_P2.54mm_Vertical, symbol Connector_Generic:Conn_01x03
- added J65: Conn_01x02, Connector_PinHeader_2.54mm:PinHeader_1x02_P2.54mm_Vertical, symbol Connector_Generic:Conn_01x02
- added R4, R5: 4k7, Resistor_SMD:R_0603_1608Metric_Pad0.98x0.95mm_HandSolder, symbol Device:R
- added R65: 10k, Resistor_SMD:R_0603_1608Metric_Pad0.98x0.95mm_HandSolder, symbol Device:R
- added U65: LTV-817S, Package_DIP:SMDIP-4_W9.53mm, symbol Isolator:LTV-817S
- C10, C11, C12: footprint Capacitor_SMD:C_0805_2012Metric_Pad1.18x1.45mm_HandSolder -> Capacitor_SMD:C_0603_1608Metric_Pad1.08x0.95mm_HandSolder; Mouser (none) -> 581-06035C104KAT2A
Connections:
- net +3V3: now also R4.2, R5.2, R65.2
- net BTN_1: now also J11.1 (Pin_1)
- net BTN_2: now also J11.2 (Pin_2)
- net GND: now also J11.3 (Pin_3), U65.3
- net I2C_SCL: now also R4.1
- net I2C_SDA: now also R5.1
- new net: J65.1 (Pin_1), U65.1
- new net: J65.2 (Pin_2), U65.2
- new net AIN_TTL: R65.1, U65.4
Other:
- moved on the sheet: J4, J5, J8, J90, JP90

Commit message: RevB first gerber export
Parts:
- added C4: 100n, Capacitor_SMD:C_0603_1608Metric_Pad1.08x0.95mm_HandSolder, symbol Device:C
- added D4: SK6812, LED_SMD:LED_SK6812_PLCC4_5.0x5.0mm_P3.2mm, symbol LED:SK6812
- added D65: PMEG60T10ELRX, Diode_SMD:D_SOD-123, symbol Device:D
- added R66: 10k, Resistor_SMD:R_0603_1608Metric_Pad0.98x0.95mm_HandSolder, symbol Device:R
Connections:
- net GPIO12 is gone; now on net AIN_TTL: J7.2 (Pin_2), U10.20 (GPIO12/TOUCH11/ADC2_CH0/FSPICS0/FSPIIO4/SUBSPICS0)
- net +3V3: now also C4.1, D4.3 (VDD)
- net GND: now also C4.2, D4.1 (VSS)
- net at J65.1 (Pin_1): now also D65.2 (A); no longer U65.1
- net at J65.2 (Pin_2): now also R66.1; no longer U65.2
- net LED_DIN: now reaches U10.31 (GPIO38/FSPIWP/SUBSPIWP)
- net LED_DIN: now also D4.2 (DIN)
- new net: R66.2, U65.2
- new net: D65.1 (K), U65.1
